File: PCB/FDC.kicad_pcb (KiCad board)
At the start: 2 copper layers, 140.3 x 97.8 mm, 27 parts, among them J1 Floppy, J2 Floopy Power Pin6, J3 EXPANSION, U1 7406, X1 8Mhz

Commit message: Added Pull-ups to WD177X
Parts:
- added R4: 1K, 8bits:R_Axial_DIN0204_L3.6mm_D1.6mm_P11.43mm_Horizontal, F.Cu at (149.9, 82.6)
- added R5: 1K, 8bits:R_Axial_DIN0204_L3.6mm_D1.6mm_P11.43mm_Horizontal, F.Cu at (147.3, 82.6)
- added R6: 1K, 8bits:R_Axial_DIN0204_L3.6mm_D1.6mm_P11.43mm_Horizontal, F.Cu at (110.5, 85.1)
- added R7: 1K, 8bits:R_Axial_DIN0204_L3.6mm_D1.6mm_P11.43mm_Horizontal, F.Cu at (108.0, 85.1)
- J3: footprint FDC:Edge_Card_Connector_22x2 -> 8bits:COMiX35_Edge_Card_Connector_22x2
- moved R3 1.27 mm to (105.4, 77.5)
- renumbered R6 to R10, R7 to R9
Routing:
- net GND: track 17.2 -> 29.3 mm, vias 4 -> 8
- net /~{IP}: track 76.0 -> 77.5 mm, vias 2 -> 1
- net /~{WPRT}: track 62.4 -> 63.7 mm
- net /~{TR00}: track 56.6 -> 57.3 mm, vias 3 -> 2
- net /Main/~{DDEN}: track 4.42 -> 4.95 mm
- net /~{RD}: track 40.9 -> 41.3 mm, vias 3 -> 2
