File: PCB/FDC.kicad_sch (KiCad schematic)
At the start: 4 parts, among them J1 Floppy, J2 Floopy Power Pin6, J3 EXPANSION

Commit message: Added Pull-ups to WD177X
Parts:
- J3: footprint Connector_PinHeader_2.54mm:PinHeader_2x22_P2.54mm_Vertical -> 8bits:COMiX35_Edge_Card_Connector_22x2
