File: PCB/Main.kicad_sch (KiCad schematic)
At the start: 23 parts, among them U1 7406, X1 8Mhz

Commit message: Added Pull-ups to WD177X
Parts:
- added R4, R5, R6, R7: 1K, 8bits:R_Axial_DIN0204_L3.6mm_D1.6mm_P11.43mm_Horizontal, symbol Device:R_US
- renumbered R6 to R10, R7 to R9
Connections:
- net +5V: now also R4.2, R5.2, R6.2, R7.2
- net ~{IP}: now also R6.1
- net ~{RD}: now also R4.1
- net ~{TR00}: now also R5.1
- net ~{WPRT}: now also R7.1
